File: hardware/StealthKitty.kicad_pro/brain.kicad_sch (KiCad schematic)
At the start: 28 parts, among them J401 Conn_ST_STDC14, SW401 SW_Push, SW402 SW_Push, U401 STM32G431CBU6, Y401 Crystal_GND24_Small

Commit message: Modif PCB 16/10/2024 V2
Parts:
- C402, C407, C410: footprint Capacitor_SMD:C_0402_1005Metric -> Capacitor_SMD:C_0603_1608Metric
Connections:
- net status_LiDar is gone; now on net status_LiDAR: D403.2 (A)
- net status_LiDAR: now reaches U401.38 (PA15)
Changed lines of the file:
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@@
 	)
 	(no_connect
-		(at 125.73 125.73)
+		(at 252.73 49.53)
 	)
 	(no_connect
-		(at 252.73 49.53)
+		(at 92.71 107.95)
 	)
 	(no_connect
@@
 	(wire
 		(pts
+			(xy 133.35 125.73) (xy 125.73 125.73)
+		)
+		(stroke
+			(width 0)
+			(type default)
+		)
+	)
+	(wire
+		(pts
 			(xy 107.95 76.2) (xy 105.41 76.2)
 		)
@@
 		)
 	)
-	(label "status_LiDar"
+	(label "status_LiDAR"
 		(at 158.75 133.35 0)
 		(fields_autoplaced yes)
@@
 		)
 	)
+	(label "status_LiDAR"
+		(at 133.35 125.73 0)
+		(fields_autoplaced yes)
+		(effects
+			(font
+				(size 1.27 1.27)
+			)
+			(justify left bottom)
+		)
+	)
 	(label "status_Orange"
 		(at 88.9 158.75 180)
@@
 			)
 		)
-		(property "Footprint" "Capacitor_SMD:C_0402_1005Metric"
+		(property "Footprint" "Capacitor_SMD:C_0603_1608Metric"
 			(at 67.31 80.01 0)
 			(effects
@@
 			)
 		)
-		(property "Footprint" "Capacitor_SMD:C_0402_1005Metric"
+		(property "Footprint" "Capacitor_SMD:C_0603_1608Metric"
 			(at 99.06 43.18 0)
 			(effects
@@
 			)
 		)
-		(property "Footprint" "Capacitor_SMD:C_0402_1005Metric"
+		(property "Footprint" "Capacitor_SMD:C_0603_1608Metric"
 			(at 140.97 80.01 0)
 			(effects

Commit message: MODIF PCB 22/10/2024
Parts:
- removed C410: 1u, Capacitor_SMD:C_0603_1608Metric, symbol Device:C_Small
- added C412: 100nF, Capacitor_SMD:C_0402_1005Metric, symbol Device:C_Small
- added R406: 10k, Resistor_SMD:R_0402_1005Metric, symbol Device:R_Small
- added R407: 10K, Resistor_SMD:R_0402_1005Metric, symbol Device:R_Small
Connections:
- net +3.3V: now also R406.1
- net Button_1: now also C412.1, R407.1; no longer SW402.1
- net GND: now also C412.2
- new net: R406.2, R407.2, SW402.1
Other:
- moved on the sheet: C408, SW402

Commit message: Modif après revue du prof le 22/10
Changed lines of the file:
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@@
 	(wire
 		(pts
-			(xy 133.35 125.73) (xy 125.73 125.73)
+			(xy 140.97 125.73) (xy 125.73 125.73)
 		)
 		(stroke
@@
 	(wire
 		(pts
-			(xy 127 95.25) (xy 125.73 95.25)
+			(xy 134.62 95.25) (xy 125.73 95.25)
 		)
 		(stroke
@@
 	(wire
 		(pts
+			(xy 125.73 92.71) (xy 134.62 92.71)
+		)
+		(stroke
+			(width 0)
+			(type default)
+		)
+	)
+	(wire
+		(pts
 			(xy 236.22 71.12) (xy 236.22 73.66)
 		)
@@
 	(wire
 		(pts
-			(xy 127 92.71) (xy 125.73 92.71)
-		)
-		(stroke
-			(width 0)
-			(type default)
-		)
-	)
-	(wire
-		(pts
 			(xy 63.5 38.1) (xy 63.5 40.64)
 		)
@@
 	(wire
 		(pts
-			(xy 63.5 48.26) (xy 59.69 48.26)
+			(xy 63.5 48.26) (xy 58.42 48.26)
 		)
 		(stroke
@@
 	(wire
 		(pts
-			(xy 125.73 113.03) (xy 143.51 113.03)
-		)
-		(stroke
-			(width 0)
-			(type default)
-		)
-	)
-	(wire
-		(pts
 			(xy 78.74 140.97) (xy 92.71 140.97)
 		)
@@
 	(wire
 		(pts
-			(xy 59.69 48.26) (xy 59.69 49.53)
+			(xy 58.42 48.26) (xy 58.42 49.53)
 		)
 		(stroke
@@
 	(wire
 		(pts
-			(xy 144.78 86.36) (xy 144.78 82.55)
+			(xy 144.78 83.82) (xy 144.78 82.55)
 		)
 		(stroke
@@
 	)
 	(label "TX_link"
-		(at 127 92.71 0)
+		(at 134.62 92.71 0)
 		(fields_autoplaced yes)
 		(effects
@@
 	)
 	(label "RX_link"
-		(at 127 95.25 0)
+		(at 134.62 95.25 0)
 		(fields_autoplaced yes)
 		(effects
@@
 	)
 	(label "status_LiDAR"
-		(at 133.35 125.73 0)
+		(at 140.97 125.73 0)
 		(fields_autoplaced yes)
 		(effects
@@
 	(global_label "M_SCTR"
 		(shape input)
-		(at 143.51 113.03 0)
+		(at 125.73 113.03 0)
 		(fields_autoplaced yes)
 		(effects
@@
 		)
 		(property "Intersheetrefs" "${INTERSHEET_REFS}"
-			(at 153.6313 113.03 0)
+			(at 135.8513 113.03 0)
 			(effects
 				(font
@@
 		(dnp no)
 		(property "Reference" "C403"
-			(at 72.39 97.282 0)
+			(at 70.612 97.028 0)
 			(effects
 				(font
@@
 		)
 		(property "Value" "100 nF"
-			(at 80.772 97.79 0)
+			(at 71.374 99.06 0)
 			(effects
 				(font
@@
 		(dnp no)
 		(property "Reference" "D401"
-			(at 180.34 97.79 0)
+			(at 180.34 96.774 0)
 			(effects
 				(font
@@
 		)
 		(property "Value" "LED_status_orange"
-			(at 180.34 100.33 0)
+			(at 180.34 99.06 0)
 			(effects
 				(font
@@
 	(symbol
 		(lib_id "power:GND")
-		(at 144.78 86.36 0)
+		(at 144.78 83.82 0)
 		(unit 1)
 		(exclude_from_sim no)
@@
 		(fields_autoplaced yes)
 		(property "Reference" "#PWR0412"
-			(at 144.78 92.71 0)
+			(at 144.78 90.17 0)
 			(effects
 				(font
@@
 		)
 		(property "Value" "GND"
-			(at 144.78 91.44 0)
+			(at 144.78 88.9 0)
 			(effects
 				(font
@@
 		)
 		(property "Footprint" ""
-			(at 144.78 86.36 0)
+			(at 144.78 83.82 0)
 			(effects
 				(font
@@
 		)
 		(property "Datasheet" ""
-			(at 144.78 86.36 0)
+			(at 144.78 83.82 0)
 			(effects
 				(font
@@
 		)
 		(property "Description" "Power symbol creates a global label with name \"GND\" , ground"
-			(at 144.78 86.36 0)
+			(at 144.78 83.82 0)
 			(effects
 				(font
@@
 		)
 		(instances
-			(project ""
+			(project "StealthKitty.kicad_pro"
 				(path "/23d5732b-7ccb-40aa-85a2-3b18421ac23b/80e324d5-3692-40e2-ae7b-7b2010b2e090"
 					(reference "#PWR0423")
@@
 		)
 		(property "Value" "100 nF"
-			(at 66.04 44.4562 0)
+			(at 65.532 44.45 0)
 			(effects
 				(font
@@
 		)
 		(property "Value" "100 nF"
-			(at 91.44 44.4562 0)
+			(at 90.932 44.704 0)
 			(effects
 				(font
@@
 		)
 		(instances
-			(project ""
+			(project "StealthKitty.kicad_pro"
 				(path "/23d5732b-7ccb-40aa-85a2-3b18421ac23b/80e324d5-3692-40e2-ae7b-7b2010b2e090"
 					(reference "R406")
@@
 		)
 		(property "Value" "10 pF"
-			(at 135.89 53.3462 0)
+			(at 135.382 53.594 0)
 			(effects
 				(font
@@
 		)
 		(property "Value" "100nF"
-			(at 231.14 138.4362 0)
+			(at 221.488 139.446 0)
 			(effects
 				(font
@@
 		(dnp no)
 		(property "Reference" "C405"
-			(at 83.82 82.042 0)
+			(at 81.026 76.962 0)
 			(effects
 				(font
@@
 		)
 		(property "Value" "100 nF"
-			(at 77.47 44.4562 0)
+			(at 76.708 44.45 0)
 			(effects
 				(font
@@
 		(dnp no)
 		(property "Reference" "C402"
-			(at 66.04 82.042 0)
+			(at 65.278 77.216 0)
 			(effects
 				(font
@@
 		)
 		(property "Value" "4.7 uF"
-			(at 101.6 44.4562 0)
+			(at 101.092 44.704 0)
 			(effects
 				(font
@@
 		(on_board yes)
 		(dnp no)
-		(fields_autoplaced yes)
 		(property "Reference" "R403"
-			(at 191.77 97.79 90)
+			(at 191.77 96.266 90)
 			(effects
 				(font
@@
 		(dnp no)
 		(property "Reference" "C408"
-			(at 143.51 82.042 0)
+			(at 141.986 78.994 0)
 			(effects
 				(font
@@
 		)
 		(property "Value" "10 nF"
-			(at 142.24 78.7338 0)
+			(at 142.494 81.28 0)
 			(effects
 				(font
@@
 		(on_board yes)
 		(dnp no)
-		(fields_autoplaced yes)
 		(property "Reference" "R401"
-			(at 39.37 154.9399 0)
+			(at 37.846 153.416 0)
 			(effects
 				(font
@@
 		)
 		(property "Value" "3.3k"
-			(at 39.37 157.4799 0)
+			(at 38.354 155.956 0)
 			(effects
 				(font
@@
 	(symbol
 		(lib_id "power:GND")
-		(at 59.69 49.53 0)
+		(at 58.42 49.53 0)
 		(unit 1)
 		(exclude_from_sim no)
@@
 		(dnp no)
 		(property "Reference" "#PWR0404"
-			(at 59.69 55.88 0)
+			(at 58.42 55.88 0)
 			(effects
 				(font
@@
 		)
 		(property "Value" "GND"
-			(at 63.246 51.054 0)
+			(at 61.976 51.054 0)
 			(effects
 				(font
@@
 		)
 		(property "Footprint" ""
-			(at 59.69 49.53 0)
+			(at 58.42 49.53 0)
 			(effects
 				(font
@@
 		)
 		(property "Datasheet" ""
-			(at 59.69 49.53 0)
+			(at 58.42 49.53 0)
 			(effects
 				(font
@@
 		)
 		(property "Description" "Power symbol creates a global label with name \"GND\" , ground"
-			(at 59.69 49.53 0)
+			(at 58.42 49.53 0)
 			(effects
 				(font

Commit message: Dernier Modif 23/10/2024
Connections:
- net status_Orange renamed status_Blue
- net status_Purple renamed status_Red
Changed lines of the file:
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@@
 		)
 	)
-	(label "status_Purple"
+	(label "status_Red"
 		(at 158.75 118.11 0)
 		(fields_autoplaced yes)
@@
 		)
 	)
-	(label "status_Orange"
+	(label "status_Blue"
 		(at 157.48 102.87 0)
 		(fields_autoplaced yes)
@@
 		)
 	)
-	(label "status_Purple"
+	(label "status_Red"
 		(at 88.9 161.29 180)
 		(fields_autoplaced yes)
@@
 		)
 	)
-	(label "status_Orange"
+	(label "status_Blue"
 		(at 88.9 158.75 180)
 		(fields_autoplaced yes)
