File: hardware/StealthKitty.kicad_pro/power.kicad_sch (KiCad schematic)
At the start: 27 parts, among them SW5 Switch, U4 MP1475DJ-LF-P

Commit message: MAJ empreintes
Parts:
- H5, H6, H7, H8: footprint (none) -> MountingHole:MountingHole_3.2mm_M3_Pad_Via
Changed lines of the file:
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@@
 			)
 		)
-		(property "Footprint" ""
+		(property "Footprint" "MountingHole:MountingHole_3.2mm_M3_Pad_Via"
 			(at 218.44 78.74 0)
 			(effects
@@
 			)
 		)
-		(property "Footprint" ""
+		(property "Footprint" "MountingHole:MountingHole_3.2mm_M3_Pad_Via"
 			(at 241.3 78.74 0)
 			(effects
@@
 		(fields_autoplaced yes)
 		(property "Reference" "U4"
-			(at 73.66 54.61 0)
+			(at 73.66 53.34 0)
 			(effects
 				(font
@@
 		)
 		(property "Value" "MP1475DJ-LF-P"
-			(at 73.66 57.15 0)
+			(at 73.66 55.88 0)
 			(effects
 				(font
@@
 			)
 		)
-		(property "Footprint" ""
+		(property "Footprint" "MountingHole:MountingHole_3.2mm_M3_Pad_Via"
 			(at 233.68 78.74 0)
 			(effects
@@
 			)
 		)
-		(property "Footprint" ""
+		(property "Footprint" "MountingHole:MountingHole_3.2mm_M3_Pad_Via"
 			(at 226.06 78.74 0)
 			(effects
