File: hardware/StealthKitty.kicad_pro/power.kicad_sch (KiCad schematic)
At the start: 23 parts, among them IC501 MP1475DJ-LF-P, SW501 Switch

Commit message: Modif PCB 16/10/2024  V1
Other:
- note added: "MP1475S!!!"
Changed lines of the file:
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@@
+		)
+	)
+	(text "MP1475S!!!"
+		(exclude_from_sim no)
+		(at 87.63 51.054 0)
+		(effects
+			(font
+				(size 1.27 1.27)
+			)
 		)
 	)

Commit message: Modif PCB 16/10/2024 V2
Parts:
- BT501: footprint Connector_JST:JST_XH_S2B-XH-A_1x02_P2.50mm_Horizontal -> Connector_JST:JST_XH_S2B-XH-A-1_1x02_P2.50mm_Horizontal
- C501, C507, C509: footprint Capacitor_SMD:C_0402_1005Metric -> Capacitor_SMD:C_0805_2012Metric
- C504, C506: footprint Capacitor_SMD:C_0402_1005Metric -> Capacitor_SMD:C_0603_1608Metric
Changed lines of the file:
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@@
 			)
 		)
-		(property "Footprint" "Capacitor_SMD:C_0402_1005Metric"
+		(property "Footprint" "Capacitor_SMD:C_0805_2012Metric"
 			(at 46.99 63.5 0)
 			(effects
@@
 			)
 		)
-		(property "Footprint" "Capacitor_SMD:C_0402_1005Metric"
+		(property "Footprint" "Capacitor_SMD:C_0805_2012Metric"
 			(at 123.19 71.12 0)
 			(effects
@@
 			)
 		)
-		(property "Footprint" "Capacitor_SMD:C_0402_1005Metric"
+		(property "Footprint" "Capacitor_SMD:C_0603_1608Metric"
 			(at 62.23 162.56 0)
 			(effects
@@
 			)
 		)
-		(property "Footprint" "Connector_JST:JST_XH_S2B-XH-A_1x02_P2.50mm_Horizontal"
+		(property "Footprint" "Connector_JST:JST_XH_S2B-XH-A-1_1x02_P2.50mm_Horizontal"
 			(at 210.82 48.006 90)
 			(effects
@@
 			)
 		)
-		(property "Footprint" "Capacitor_SMD:C_0402_1005Metric"
+		(property "Footprint" "Capacitor_SMD:C_0603_1608Metric"
 			(at 101.6 166.37 0)
 			(effects
@@
 			)
 		)
-		(property "Footprint" "Capacitor_SMD:C_0402_1005Metric"
+		(property "Footprint" "Capacitor_SMD:C_0805_2012Metric"
 			(at 111.76 71.12 0)
 			(effects

Commit message: Modif après revue du prof le 22/10
Changed lines of the file:
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@@
 	(wire
 		(pts
+			(xy 50.8 81.28) (xy 50.8 80.01)
+		)
+		(stroke
+			(width 0)
+			(type default)
+		)
+	)
+	(wire
+		(pts
 			(xy 248.92 46.99) (xy 252.73 46.99)
 		)
@@
 	(wire
 		(pts
-			(xy 92.71 66.04) (xy 96.52 66.04)
-		)
-		(stroke
-			(width 0)
-			(type default)
-		)
-	)
-	(wire
-		(pts
 			(xy 100.33 88.9) (xy 100.33 77.47)
 		)
@@
 	(wire
 		(pts
-			(xy 177.8 143.51) (xy 181.61 143.51)
+			(xy 175.26 143.51) (xy 181.61 143.51)
 		)
 		(stroke
@@
 	(wire
 		(pts
-			(xy 87.63 64.77) (xy 92.71 64.77)
+			(xy 234.95 46.99) (xy 248.92 46.99)
 		)
 		(stroke
@@
 	(wire
 		(pts
-			(xy 234.95 46.99) (xy 248.92 46.99)
+			(xy 127 66.04) (xy 127 88.9)
 		)
 		(stroke
@@
 	(wire
 		(pts
-			(xy 127 66.04) (xy 127 88.9)
+			(xy 87.63 66.04) (xy 96.52 66.04)
+		)
+		(stroke
+			(width 0)
+			(type default)
+		)
+	)
+	(wire
+		(pts
+			(xy 87.63 66.04) (xy 87.63 64.77)
 		)
 		(stroke
@@
 	(wire
 		(pts
-			(xy 92.71 64.77) (xy 92.71 66.04)
-		)
-		(stroke
-			(width 0)
-			(type default)
-		)
-	)
-	(wire
-		(pts
 			(xy 210.82 53.34) (xy 210.82 52.07)
 		)
@@
 	(symbol
 		(lib_id "power:GND")
-		(at 50.8 80.01 0)
+		(at 50.8 81.28 0)
 		(unit 1)
 		(exclude_from_sim no)
@@
 		(dnp no)
 		(property "Reference" "#PWR0503"
-			(at 50.8 86.36 0)
+			(at 50.8 87.63 0)
 			(effects
 				(font
@@
 		)
 		(property "Value" "GND"
-			(at 48.26 82.55 0)
+			(at 47.244 82.55 0)
 			(effects
 				(font
@@
 		)
 		(property "Footprint" ""
-			(at 50.8 80.01 0)
+			(at 50.8 81.28 0)
 			(effects
 				(font
@@
 		)
 		(property "Datasheet" ""
-			(at 50.8 80.01 0)
+			(at 50.8 81.28 0)
 			(effects
 				(font
@@
 		)
 		(property "Description" ""
-			(at 50.8 80.01 0)
+			(at 50.8 81.28 0)
 			(effects
 				(font
@@
 		)
 		(property "Value" "100k"
-			(at 19.05 64.77 0)
+			(at 19.05 64.262 0)
 			(effects
 				(font
@@
 		(dnp no)
 		(property "Reference" "C501"
-			(at 45.72 64.77 0)
+			(at 44.958 62.23 0)
 			(effects
 				(font
@@
 		)
 		(property "Value" "22uF"
-			(at 45.72 62.23 0)
+			(at 44.704 65.024 0)
 			(effects
 				(font
@@
 		(on_board yes)
 		(dnp no)
-		(fields_autoplaced yes)
 		(property "Reference" "C509"
-			(at 120.65 71.7614 0)
+			(at 120.396 70.358 0)
 			(effects
 				(font
@@
 		)
 		(property "Value" "22uF"
-			(at 120.65 69.2214 0)
+			(at 120.65 72.0154 0)
 			(effects
 				(font
@@
 		(dnp no)
 		(property "Reference" "L501"
-			(at 105.41 60.96 90)
+			(at 106.172 60.706 90)
 			(effects
 				(font
@@
 		)
 		(property "Value" "4.7uH"
-			(at 105.41 63.5 90)
+			(at 106.172 63.246 90)
 			(effects
 				(font
@@
 		(dnp no)
 		(property "Reference" "C505"
-			(at 87.63 63.5 0)
+			(at 89.408 63.246 0)
 			(effects
 				(font
@@
 		)
 		(property "Value" "0.1uF"
-			(at 87.63 64.77 0)
+			(at 89.408 64.77 0)
 			(effects
 				(font
@@
 		(on_board yes)
 		(dnp no)
-		(fields_autoplaced yes)
 		(property "Reference" "R504"
 			(at 97.79 72.39 90)
@@
 		)
 		(property "Value" "16k"
-			(at 97.79 74.93 90)
+			(at 97.536 75.184 90)
 			(effects
 				(font
@@
 		(on_board yes)
 		(dnp no)
-		(fields_autoplaced yes)
 		(property "Reference" "C507"
-			(at 109.22 71.7614 0)
+			(at 109.22 70.358 0)
 			(effects
 				(font
@@
 		)
 		(property "Value" "22uF"
-			(at 109.22 69.2214 0)
+			(at 109.22 72.0154 0)
 			(effects
 				(font
@@
 	(symbol
 		(lib_id "power:+3.3V")
-		(at 177.8 143.51 0)
+		(at 175.26 143.51 0)
 		(unit 1)
 		(exclude_from_sim no)
@@
 		(fields_autoplaced yes)
 		(property "Reference" "#PWR0513"
-			(at 177.8 147.32 0)
+			(at 175.26 147.32 0)
 			(effects
 				(font
@@
 		)
 		(property "Value" "+3.3V"
-			(at 177.8 138.43 0)
+			(at 175.26 138.43 0)
 			(effects
 				(font
@@
 		)
 		(property "Footprint" ""
-			(at 177.8 143.51 0)
+			(at 175.26 143.51 0)
 			(effects
 				(font
@@
 		)
 		(property "Datasheet" ""
-			(at 177.8 143.51 0)
+			(at 175.26 143.51 0)
 			(effects
 				(font
@@
 		)
 		(property "Description" "Power symbol creates a global label with name \"+3.3V\""
-			(at 177.8 143.51 0)
+			(at 175.26 143.51 0)
 			(effects
 				(font
@@
 		(dnp no)
 		(property "Reference" "C503"
-			(at 56.896 64.516 0)
+			(at 58.166 61.976 0)
 			(effects
 				(font
@@
 		)
 		(property "Value" "0.1uF"
-			(at 58.42 62.23 0)
+			(at 58.166 65.278 0)
 			(effects
 				(font
