File: hardware/StealthKitty.kicad_pro/sensor.kicad_sch (KiCad schematic)
At the start: 13 parts, among them J301 Conn_01x06, J302 Conn_01x06, J303 Conn_01x08, U301 ADXL343

Commit message: Modif Routage V2
Parts:
- removed TP305: TestPoint, TestPoint:TestPoint_Pad_D1.5mm, symbol Connector:TestPoint
Changed lines of the file:
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@@
-	)
-	(junction
-		(at 102.87 36.83)
-		(diameter 0)
-		(color 0 0 0 0)
 	)
 	(junction
@@
 	(wire
 		(pts
-			(xy 50.8 36.83) (xy 50.8 40.64)
-		)
-		(stroke
-			(width 0)
-			(type default)
-		)
-	)
-	(wire
-		(pts
-			(xy 31.75 45.72) (xy 52.07 45.72)
+			(xy 49.53 39.37) (xy 58.42 39.37)
 		)
 		(stroke
@@
 	(wire
 		(pts
-			(xy 50.8 36.83) (xy 58.42 36.83)
-		)
-		(stroke
-			(width 0)
-			(type default)
-		)
-	)
-	(wire
-		(pts
 			(xy 142.24 105.41) (xy 152.4 105.41)
 		)
@@
 		)
 	)
-	(wire
-		(pts
-			(xy 118.11 41.91) (xy 118.11 39.37)
-		)
-		(stroke
-			(width 0)
-			(type default)
-		)
-	)
 	(polyline
 		(pts
@@
 	(wire
 		(pts
-			(xy 31.75 40.64) (xy 50.8 40.64)
+			(xy 39.37 36.83) (xy 58.42 36.83)
 		)
 		(stroke
@@
 	(wire
 		(pts
-			(xy 52.07 39.37) (xy 52.07 45.72)
-		)
-		(stroke
-			(width 0)
-			(type default)
-		)
-	)
-	(wire
-		(pts
 			(xy 45.72 31.75) (xy 58.42 31.75)
 		)
@@
 	(wire
 		(pts
-			(xy 102.87 36.83) (xy 123.19 36.83)
+			(xy 99.06 36.83) (xy 123.19 36.83)
 		)
 		(stroke
@@
 	(wire
 		(pts
-			(xy 99.06 36.83) (xy 102.87 36.83)
-		)
-		(stroke
-			(width 0)
-			(type default)
-		)
-	)
-	(wire
-		(pts
 			(xy 110.49 29.21) (xy 110.49 34.29)
 		)
@@
 	(wire
 		(pts
-			(xy 52.07 39.37) (xy 58.42 39.37)
-		)
-		(stroke
-			(width 0)
-			(type default)
-		)
-	)
-	(wire
-		(pts
-			(xy 102.87 33.02) (xy 102.87 36.83)
-		)
-		(stroke
-			(width 0)
-			(type default)
-		)
-	)
-	(wire
-		(pts
-			(xy 99.06 41.91) (xy 118.11 41.91)
-		)
-		(stroke
-			(width 0)
-			(type default)
-		)
-	)
-	(wire
-		(pts
-			(xy 118.11 39.37) (xy 123.19 39.37)
+			(xy 110.49 39.37) (xy 123.19 39.37)
 		)
 		(stroke
@@
 	(global_label "INT_tof1"
 		(shape input)
-		(at 31.75 40.64 180)
+		(at 39.37 36.83 180)
 		(fields_autoplaced yes)
 		(effects
@@
 		)
 		(property "Intersheetrefs" "${INTERSHEET_REFS}"
-			(at 21.0844 40.64 0)
+			(at 28.7044 36.83 0)
 			(effects
 				(font
@@
 	(global_label "xshunt1"
 		(shape input)
-		(at 31.75 45.72 180)
+		(at 49.53 39.37 180)
 		(fields_autoplaced yes)
 		(effects
@@
 		)
 		(property "Intersheetrefs" "${INTERSHEET_REFS}"
-			(at 21.3264 45.72 0)
+			(at 39.1064 39.37 0)
 			(effects
 				(font
@@
 	(global_label "xshunt2"
 		(shape input)
-		(at 99.06 41.91 180)
+		(at 110.49 39.37 180)
 		(fields_autoplaced yes)
 		(effects
@@
 		)
 		(property "Intersheetrefs" "${INTERSHEET_REFS}"
-			(at 89.8459 41.91 0)
+			(at 101.2759 39.37 0)
 			(effects
 				(font
@@
 					(unit 1)
 				)
-			)
-		)
-	)
-	(symbol
-		(lib_id "Connector:TestPoint")
-		(at 102.87 33.02 0)
-		(unit 1)
-		(exclude_from_sim no)
-		(in_bom yes)
-		(on_board yes)
-		(dnp no)
-		(property "Reference" "TP305"
-			(at 98.298 28.448 0)
-			(effects
-				(font
-					(size 1.27 1.27)
-				)
-				(justify left)
-			)
-		)
-		(property "Value" "TestPoint"
-			(at 92.964 30.988 0)
-			(effects
-				(font
-					(size 1.27 1.27)
-				)
-				(justify left)
-			)
-		)
-		(property "Footprint" "TestPoint:TestPoint_Pad_D1.5mm"
-			(at 107.95 33.02 0)
-			(effects
-				(font
-					(size 1.27 1.27)
-				)
-				(hide yes)
-			)
-		)
-		(property "Datasheet" "~"
-			(at 107.95 33.02 0)
-			(effects
-				(font
-					(size 1.27 1.27)
-				)
-				(hide yes)
-			)
-		)
-		(property "Description" "test point"
-			(at 102.87 33.02 0)
-			(effects
-				(font
-					(size 1.27 1.27)
-				)
-				(hide yes)
-			)
-		)
-		(pin "1"
-		)
-		(instances
-			(project "StealthKitty.kicad_pro"
-				(path "/23d5732b-7ccb-40aa-85a2-3b18421ac23b/8cd8413a-9ba4-4bd6-b413-2331caa50cc2"
-					(reference "TP305")
-					(unit 1)
-				)

Commit message: Modif PCB 16/10/2024 V2
Parts:
- Cs301: footprint Capacitor_SMD:C_0402_1005Metric -> Capacitor_SMD:C_0603_1608Metric
Changed lines of the file:
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@@
 			)
 		)
-		(property "Footprint" "Capacitor_SMD:C_0402_1005Metric"
+		(property "Footprint" "Capacitor_SMD:C_0603_1608Metric"
 			(at 125.73 109.22 0)
 			(effects

Commit message: Modif après revue du prof le 22/10
Changed lines of the file:
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@@
 	(polyline
 		(pts
-			(xy 144.78 76.2) (xy 284.48 76.2)
+			(xy 143.51 76.2) (xy 284.48 76.2)
 		)
 		(stroke
@@
 	(wire
 		(pts
+			(xy 189.23 52.07) (xy 212.09 52.07)
+		)
+		(stroke
+			(width 0)
+			(type default)
+		)
+	)
+	(wire
+		(pts
 			(xy 156.21 139.7) (xy 149.86 139.7)
 		)
@@
 	(polyline
 		(pts
-			(xy 12.7 76.2) (xy 144.78 76.2)
+			(xy 12.7 76.2) (xy 143.51 76.2)
 		)
 		(stroke
@@
 	(wire
 		(pts
-			(xy 110.49 34.29) (xy 123.19 34.29)
+			(xy 106.68 34.29) (xy 123.19 34.29)
 		)
 		(stroke
@@
 	(wire
 		(pts
-			(xy 99.06 36.83) (xy 123.19 36.83)
-		)
-		(stroke
-			(width 0)
-			(type default)
-		)
-	)
-	(wire
-		(pts
-			(xy 115.57 31.75) (xy 123.19 31.75)
-		)
-		(stroke
-			(width 0)
-			(type default)
-		)
-	)
-	(wire
-		(pts
-			(xy 115.57 29.21) (xy 115.57 31.75)
+			(xy 101.6 36.83) (xy 123.19 36.83)
+		)
+		(stroke
+			(width 0)
+			(type default)
+		)
+	)
+	(wire
+		(pts
+			(xy 111.76 31.75) (xy 123.19 31.75)
+		)
+		(stroke
+			(width 0)
+			(type default)
+		)
+	)
+	(wire
+		(pts
+			(xy 111.76 27.94) (xy 111.76 31.75)
 		)
 		(stroke
@@
 	(wire
 		(pts
-			(xy 110.49 29.21) (xy 110.49 34.29)
+			(xy 106.68 27.94) (xy 106.68 34.29)
 		)
 		(stroke
@@
 	(wire
 		(pts
-			(xy 110.49 39.37) (xy 123.19 39.37)
+			(xy 111.76 39.37) (xy 123.19 39.37)
 		)
 		(stroke
@@
 	(polyline
 		(pts
-			(xy 144.78 12.7) (xy 144.78 76.2)
+			(xy 143.51 12.7) (xy 143.51 76.2)
 		)
 		(stroke
@@
 	(wire
 		(pts
-			(xy 195.58 52.07) (xy 212.09 52.07)
-		)
-		(stroke
-			(width 0)
-			(type default)
-		)
-	)
-	(wire
-		(pts
 			(xy 142.24 102.87) (xy 142.24 105.41)
+		)
+		(stroke
+			(width 0)
+			(type default)
+		)
+	)
+	(wire
+		(pts
+			(xy 119.38 29.21) (xy 123.19 29.21)
 		)
 		(stroke
@@
 	(global_label "SCL"
 		(shape input)
-		(at 110.49 29.21 90)
+		(at 106.68 27.94 90)
 		(fields_autoplaced yes)
 		(effects
@@
 		)
 		(property "Intersheetrefs" "${INTERSHEET_REFS}"
-			(at 110.49 22.7172 90)
+			(at 106.68 21.4472 90)
 			(effects
 				(font
@@
 	(global_label "xshunt2"
 		(shape input)
-		(at 110.49 39.37 180)
+		(at 111.76 39.37 180)
 		(fields_autoplaced yes)
 		(effects
@@
 		)
 		(property "Intersheetrefs" "${INTERSHEET_REFS}"
-			(at 101.2759 39.37 0)
+			(at 102.5459 39.37 0)
 			(effects
 				(font
@@
 	(global_label "INT_tof2"
 		(shape input)
-		(at 99.06 36.83 180)
+		(at 101.6 36.83 180)
 		(fields_autoplaced yes)
 		(effects
@@
 		)
 		(property "Intersheetrefs" "${INTERSHEET_REFS}"
-			(at 88.3944 36.83 0)
+			(at 90.9344 36.83 0)
 			(effects
 				(font
@@
 	(global_label "SDA"
 		(shape input)
-		(at 115.57 29.21 90)
+		(at 111.76 27.94 90)
 		(fields_autoplaced yes)
 		(effects
@@
 		)
 		(property "Intersheetrefs" "${INTERSHEET_REFS}"
-			(at 115.57 22.6567 90)
+			(at 111.76 21.3867 90)
 			(effects
 				(font
@@
 		)
 		(property "Value" "TestPoint"
-			(at 127.5146 153.2457 0)
+			(at 123.698 153.162 0)
 			(effects
 				(font
@@
 		(on_board yes)
 		(dnp no)
-		(fields_autoplaced yes)
 		(property "Reference" "J302"
-			(at 130.81 34.2899 0)
+			(at 132.334 34.29 0)
 			(effects
 				(font
@@
 	(symbol
 		(lib_id "power:+5V")
-		(at 195.58 52.07 0)
+		(at 189.23 52.07 0)
 		(unit 1)
 		(exclude_from_sim no)
@@
 		(on_board yes)
 		(dnp no)
-		(fields_autoplaced yes)
 		(property "Reference" "#PWR0311"
-			(at 195.58 55.88 0)
+			(at 189.23 55.88 0)
 			(effects
 				(font
@@
 		)
 		(property "Value" "+5V"
-			(at 195.58 46.99 0)
+			(at 186.69 50.038 0)
 			(effects
 				(font
@@
 		)
 		(property "Footprint" ""
-			(at 195.58 52.07 0)
+			(at 189.23 52.07 0)
 			(effects
 				(font
@@
 		)
 		(property "Datasheet" ""
-			(at 195.58 52.07 0)
+			(at 189.23 52.07 0)
 			(effects
 				(font
@@
 		)
 		(property "Description" "Power symbol creates a global label with name \"+5V\""
-			(at 195.58 52.07 0)
+			(at 189.23 52.07 0)
 			(effects
 				(font
@@
 	(symbol
 		(lib_id "power:+5V")
-		(at 123.19 29.21 0)
+		(at 119.38 29.21 0)
 		(unit 1)
 		(exclude_from_sim no)
@@
 		(on_board yes)
 		(dnp no)
-		(fields_autoplaced yes)
 		(property "Reference" "#PWR0303"
-			(at 123.19 33.02 0)
+			(at 119.38 33.02 0)
 			(effects
 				(font
@@
 		)
 		(property "Value" "+5V"
-			(at 123.19 24.13 0)
+			(at 121.666 27.94 0)
 			(effects
 				(font
@@
 		)
 		(property "Footprint" ""
-			(at 123.19 29.21 0)
+			(at 119.38 29.21 0)
 			(effects
 				(font
@@
 		)
 		(property "Datasheet" ""
-			(at 123.19 29.21 0)
+			(at 119.38 29.21 0)
 			(effects
 				(font
@@
 		)
 		(property "Description" "Power symbol creates a global label with name \"+5V\""
-			(at 123.19 29.21 0)
+			(at 119.38 29.21 0)
 			(effects
 				(font
@@
 		(on_board yes)
 		(dnp no)
-		(fields_autoplaced yes)
 		(property "Reference" "#PWR0310"
 			(at 189.23 50.8 0)
@@
 		)
 		(property "Value" "GND"
-			(at 189.23 49.53 0)
+			(at 187.198 44.196 0)
 			(effects
 				(font
@@
 		(on_board yes)
 		(dnp no)
-		(fields_autoplaced yes)
 		(property "Reference" "U301"
-			(at 152.4 130.8414 0)
+			(at 150.622 127 0)
 			(effects
 				(font
@@
 		)
 		(property "Value" "ADXL343"
-			(at 152.4 133.3814 0)
+			(at 151.638 130.302 0)
 			(effects
 				(font
@@
 		(on_board yes)
 		(dnp no)
-		(fields_autoplaced yes)
 		(property "Reference" "J301"
-			(at 66.04 34.2899 0)
+			(at 66.802 34.29 0)
 			(effects
 				(font
@@
 		)
 		(property "Value" "Conn_01x06"
-			(at 66.04 36.8299 0)
+			(at 65.532 36.83 0)
 			(effects
 				(font
@@
 		)
 		(property "Value" "TestPoint"
-			(at 130.048 149.098 0)
+			(at 126.238 148.336 0)
 			(effects
 				(font
@@
 		)
 		(property "Value" "TestPoint"
-			(at 123.698 166.878 0)
-			(effects
-				(font
+			(at 119.126 167.132 0)
+			(effects
+				(font
