File: hardware/StealthKitty.kicad_pro/_autosave-StealthKitty.kicad_pro.kicad_pcb (KiCad board)
At the start: 4 copper layers, 53.9 x 57 mm, 77 parts, among them IC501 MP1475DJ-LF-P, J201 Conn_01x06, J202 Conn_01x06, J302 Conn_01x06, SW501 Switch, U301 ADXL343, U401 STM32G431CBU6

Commit message: Modif PCB 16/10/2024  V1
Parts:
- moved PWM2 CH1 1.60 mm to (143.6, 108.0)
Routing:
- net +VBAT: track 8.82 -> 10.9 mm, vias 7 -> 9
- net Net-(BT501-+): track 11.9 -> 13.4 mm
- net +5V: track 85.4 -> 86.4 mm
